File: Microtus-rp2040.sch (KiCad schematic (older format))
At the start: 36 parts, among them J1 Conn_01x04, J2 USB_C_Receptacle_USB2.0, SW1 SW_Push, SW3 SW_Push, SW4 SW_SPST, SW5 Rotary_Encoder, U1 AMS1117-3.3, U2 W25Q128JVS, U3 USBLC6-2SC6, U4 RP2040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

Commit message: moving things around
Changed lines of the file:
@@
 F 2 "sparkfun-sw:JOYSTICK" H 9200 4050 20  0001 C CNN
 F 3 "" H 9200 3400 50  0001 C CNN
-F 4 "COMP-09744" H 9478 3266 60  0000 L CNN "Field4"
+F 4 "COMP-09744" H 9478 3266 60  0001 L CNN "Field4"
 	1    9200 3400
 	1    0    0    -1
